Commit message: add dsr_gazebo2(m1013)

File: dsr_description2/urdf/a0509.urdf (robot description, URDF)
Before this commit: robot a0509, 8 links, 7 joints
Links:
- link base_0: geometry visual mesh filename=package://dsr_description2/meshes/a0509_white/A0509_0_0.dae scale=0.001 0.001 0.001
- link link1: geometry visual mesh filename=package://dsr_description2/meshes/a0509_white/A0509_1_0.dae scale=0.001 0.001 0.001; visual mesh filename=package://dsr_description2/meshes/a0509_white/A0509_1_1.dae scale=0.001 0.001 0.001
- link link2: geometry visual mesh filename=package://dsr_description2/meshes/a0509_white/A0509_2_0.dae scale=0.001 0.001 0.001; visual mesh filename=package://dsr_description2/meshes/a0509_white/A0509_2_1.dae scale=0.001 0.001 0.001
- link link3: geometry visual mesh filename=package://dsr_description2/meshes/a0509_white/A0509_3_0.dae scale=0.001 0.001 0.001; visual mesh filename=package://dsr_description2/meshes/a0509_white/A0509_3_1.dae scale=0.001 0.001 0.001
- link link4: geometry visual mesh filename=package://dsr_description2/meshes/a0509_white/A0509_4_0.dae scale=0.001 0.001 0.001; visual mesh filename=package://dsr_description2/meshes/a0509_white/A0509_4_1.dae scale=0.001 0.001 0.001
- link link5: geometry visual mesh filename=package://dsr_description2/meshes/a0509_white/A0509_5_0.dae scale=0.001 0.001 0.001; visual mesh filename=package://dsr_description2/meshes/a0509_white/A0509_5_1.dae scale=0.001 0.001 0.001
- link link6: geometry visual mesh filename=package://dsr_description2/meshes/a0509_white/A0509_6_0.dae scale=0.001 0.001 0.001
Joints:
- joint joint1: limit lower=-6.283 upper=6.283 effort=3460 velocity=2.094 -> lower=-2.617 upper=2.617 effort=30 velocity=1.571
- joint joint2: limit lower=-1.658 upper=1.658 effort=3460 velocity=2.094 -> lower=-2.617 upper=2.617 effort=30 velocity=1.571
- joint joint3: limit lower=-2.356 upper=2.356 effort=1630 velocity=3.142 -> lower=-2.617 upper=2.617 effort=30 velocity=1.571
- joint joint4: limit lower=-6.283 upper=6.283 effort=50 velocity=3.927 -> lower=-2.617 upper=2.617 effort=30 velocity=1.571
- joint joint5: limit lower=-2.356 upper=2.356 effort=50 velocity=3.927 -> lower=-2.617 upper=2.617 effort=30 velocity=1.571
- joint joint6: limit lower=-6.283 upper=6.283 effort=50 velocity=3.927 -> lower=-2.617 upper=2.617 effort=30 velocity=1.571

File: dsr_description2/urdf/a0912.urdf (robot description, URDF)
Before this commit: robot m0609, 8 links, 7 joints
Links:
- link link3: geometry visual mesh filename=package://dsr_description2/meshes/a0912_white/A0912_3_0.dae scale=0.001 0.001 0.001; visual mesh filename=package://dsr_description2/meshes/a0912_white/A0912_3_1.dae scale=0.001 0.001 0.001
